Commit message: some progress
Co-authored-by: Copilot <copilot@github.com>

File: src/search_rescue_robot/urdf/robot.urdf (robot description, URDF)
Before this commit: robot rescue_rover_a2, 7 links, 6 joints
Joints:
- joint camera_joint: limit lower=-0.30 upper=0.30 effort=1.2 velocity=0.9 -> lower=-0.174533 upper=0.174533 effort=1.2 velocity=0.9
