Commit message: urdf created

File: src/search_rescue_robot/urdf/robot.urdf (robot description, URDF)
Before this commit: robot rescue_rover_a2, 7 links, 6 joints
Links:
- link base_link: mass 4.8 -> 5.0; geometry collision box size=0.4 0.3 0.15; visual box size=0.4 0.3 0.15
- link camera_link: mass 0.10 -> 0.1; geometry collision box size=0.05 0.04 0.03; visual box size=0.05 0.04 0.03
- link caster_wheel: mass 0.12 -> 0.1; geometry collision sphere radius=0.025; visual sphere radius=0.025
- link left_wheel: mass 0.34 -> 0.3; geometry collision cylinder length=0.03 radius=0.075; visual cylinder length=0.03 radius=0.075
- link lidar_link: mass 0.18 -> 0.15; geometry collision cylinder length=0.03 radius=0.035; visual cylinder length=0.03 radius=0.035
- link right_wheel: mass 0.34 -> 0.3; geometry collision cylinder length=0.03 radius=0.075; visual cylinder length=0.03 radius=0.075
Joints:
- joint camera_joint: limit lower=-0.174533 upper=0.174533 effort=1.2 velocity=0.9 -> lower=-0.2618 upper=0.2618 effort=1.0 velocity=1.0; origin xyz=0.125 0 0.09 rpy=0 0 0 -> xyz=0.2 0 0.12 rpy=0 0 0
- joint caster_joint: origin xyz=0.115 0 0.028 rpy=0 0 0 -> xyz=0.15 0 0.025 rpy=0 0 0
- joint imu_joint: origin xyz=0.0 0 0.066 rpy=0 0 0 -> xyz=0 0 0.085 rpy=0 0 0
- joint left_wheel_joint: origin xyz=-0.06 0.102 0.07 rpy=0 0 0 -> xyz=-0.05 0.165 0.075 rpy=0 0 0
- joint lidar_joint: origin xyz=-0.085 0 0.14 rpy=0 0 0 -> xyz=0 0 0.165 rpy=0 0 0
- joint right_wheel_joint: origin xyz=-0.06 -0.102 0.07 rpy=0 0 0 -> xyz=-0.05 -0.165 0.075 rpy=0 0 0
